File: PCB/Star Tracker.kicad_pcb (KiCad board)
At the start: 2 copper layers, 0 parts

Commit message: Fixed broken schematic and started on layout
Parts:
- added 0.01uf1: C, Capacitor_SMD:C_1206_3216Metric, F.Cu at (131.3, 106.5)
- added 100nf1: C, Capacitor_SMD:C_1206_3216Metric, F.Cu at (131.3, 109.8)
- added 100nf2: C, Capacitor_SMD:C_1206_3216Metric, F.Cu at (136.9, 108.5)
- added 100nf3: C, Capacitor_SMD:C_1206_3216Metric, F.Cu at (177.9, 77.3)
- added 10uf1: C, Capacitor_SMD:C_1206_3216Metric, F.Cu at (142.6, 108.5)
- added 10uf2: C, Capacitor_SMD:C_1206_3216Metric, F.Cu at (148.3, 101.7)
- added 10uf3: C, Capacitor_SMD:C_1206_3216Metric, F.Cu at (153.9, 101.7)
- added 150uf1: C, Capacitor_SMD:C_1206_3216Metric, F.Cu at (148.3, 105.0)
- added 150uf2: C, Capacitor_SMD:C_1206_3216Metric, F.Cu at (148.2, 108.5)
- added 1uf1: C, Capacitor_SMD:C_1206_3216Metric, F.Cu at (177.9, 80.6)
- added 1uf2: C, Capacitor_SMD:C_1206_3216Metric, F.Cu at (167.5, 101.2)
- added 1uf3: C, Capacitor_SMD:C_1206_3216Metric, F.Cu at (177.9, 83.9)
- added 1uf4: C, Capacitor_SMD:C_1206_3216Metric, F.Cu at (153.8, 108.3)
- added 2.2uf1: C, Capacitor_SMD:C_1206_3216Metric, F.Cu at (153.9, 105.0)
- added 300k1: R, Resistor_SMD:R_1206_3216Metric, F.Cu at (159.5, 101.7)
- added 330Ohm1: R, Resistor_SMD:R_1206_3216Metric, F.Cu at (179.1, 87.2)
- added 4.7kOhm1: R, Resistor_SMD:R_1206_3216Metric, F.Cu at (159.5, 105.0)
- added 5.6pf1: C, Capacitor_SMD:C_1206_3216Metric, F.Cu at (159.4, 108.3)
- added 93k1: R, Resistor_SMD:R_1206_3216Metric, F.Cu at (165.2, 104.5)
- added IR_LED1: Screw_Terminal_01x02, Connector_Phoenix_MC:PhoenixContact_MC_1,5_2-G-3.5_1x02_P3.50mm_Horizontal, F.Cu at (157.7, 91.0)
- added J1: Conn_ARM_JTAG_SWD_10, Connector_PinHeader_1.27mm:PinHeader_2x05_P1.27mm_Vertical_SMD, F.Cu at (123.7, 104.5)
- added PWR1: Screw_Terminal_01x04, Connector_Phoenix_MC:PhoenixContact_MC_1,5_4-G-3.5_1x04_P3.50mm_Horizontal, F.Cu at (143.5, 78.9)
- added RotaryEncoder1: Screw_Terminal_01x05, Connector_Phoenix_MC:PhoenixContact_MC_1,5_5-G-3.5_1x05_P3.50mm_Horizontal, F.Cu at (122.5, 78.9)
- added Screen1: Screw_Terminal_01x04, Connector_Phoenix_MC:PhoenixContact_MC_1,5_4-G-3.5_1x04_P3.50mm_Horizontal, F.Cu at (140.2, 91.0)
- added StepperMotor1: Screw_Terminal_01x04, Connector_Phoenix_MC:PhoenixContact_MC_1,5_4-G-3.5_1x04_P3.50mm_Horizontal, F.Cu at (161.1, 78.9)
- added U1: NCV565D2TG-ND, Package_TO_SOT_SMD:TO-263-5_TabPin6, F.Cu at (127.7, 94.1)
- added U2: DRV8833PW, Package_SO:TSSOP-16_4.4x5mm_P0.65mm, F.Cu at (141.0, 103.5)
- added U3: ATSAMD21E18A-AU, Package_QFP:TQFP-32_7x7mm_P0.8mm, F.Cu at (170.5, 93.7)
- added U4: AP7312-1833W6-7, Package_TO_SOT_SMD:SOT-23-6_Handsoldering, F.Cu at (131.5, 102.6)
